Commit message: auto added

File: src/mobile_description/urdf/mobile.xacro (robot description, xacro)
@@ -156,5 +156,5 @@
   <axis xyz="0.0 -1.0 0.0"/>
 </joint>
-<joint name="Revolute 3" type="continuous"
+<joint name="Revolute 3" type="continuous">
   <origin xyz="0.145 0.17 0.0625" rpy="0 0 0"/>
   <parent link="base_link"/>

Commit message: auto added

File: src/mobile_description/urdf/mobile.xacro (robot description, xacro)
@@ -13,5 +13,5 @@
     <origin xyz="0 0 0" rpy="0 0 0"/>
     <geometry>
-      <mesh filename="package://mobile_description/meshes/base_link.stl" scale="0.001 0.001 0.001"/>
+      <mesh filename="file://$(find mobile_description)/meshes/base_link.stl" scale="0.001 0.001 0.001"/>
     </geometry>
     <material name="silver"/>
@@ -20,5 +20,5 @@
     <origin xyz="0 0 0" rpy="0 0 0"/>
     <geometry>
-      <mesh filename="package://mobile_description/meshes/base_link.stl" scale="0.001 0.001 0.001"/>
+      <mesh filename="file://$(find mobile_description)/meshes/base_link.stl" scale="0.001 0.001 0.001"/>
     </geometry>
   </collision>
@@ -33,5 +33,5 @@
     <origin xyz="0.145 0.17 -0.0625" rpy="0 0 0"/>
     <geometry>
-      <mesh filename="package://mobile_description/meshes/rear_right_wheel_1.stl" scale="0.001 0.001 0.001"/>
+      <mesh filename="file://$(find mobile_description)/meshes/rear_right_wheel_1.stl" scale="0.001 0.001 0.001"/>
     </geometry>
     <material name="silver"/>
@@ -40,5 +40,5 @@
     <origin xyz="0.145 0.17 -0.0625" rpy="0 0 0"/>
     <geometry>
-      <mesh filename="package://mobile_description/meshes/rear_right_wheel_1.stl" scale="0.001 0.001 0.001"/>
+      <mesh filename="file://$(find mobile_description)/meshes/rear_right_wheel_1.stl" scale="0.001 0.001 0.001"/>
     </geometry>
   </collision>
@@ -53,5 +53,5 @@
     <origin xyz="-0.145 0.17 -0.0625" rpy="0 0 0"/>
     <geometry>
-      <mesh filename="package://mobile_description/meshes/front_right_wheel_1.stl" scale="0.001 0.001 0.001"/>
+      <mesh filename="file://$(find mobile_description)/meshes/front_right_wheel_1.stl" scale="0.001 0.001 0.001"/>
     </geometry>
     <material name="silver"/>
@@ -60,5 +60,5 @@
     <origin xyz="-0.145 0.17 -0.0625" rpy="0 0 0"/>
     <geometry>
-      <mesh filename="package://mobile_description/meshes/front_right_wheel_1.stl" scale="0.001 0.001 0.001"/>
+      <mesh filename="file://$(find mobile_description)/meshes/front_right_wheel_1.stl" scale="0.001 0.001 0.001"/>
     </geometry>
   </collision>
@@ -73,5 +73,5 @@
     <origin xyz="-0.145 -0.17 -0.0625" rpy="0 0 0"/>
     <geometry>
-      <mesh filename="package://mobile_description/meshes/front_left_wheel_1.stl" scale="0.001 0.001 0.001"/>
+      <mesh filename="file://$(find mobile_description)/meshes/front_left_wheel_1.stl" scale="0.001 0.001 0.001"/>
     </geometry>
     <material name="silver"/>
@@ -80,5 +80,5 @@
     <origin xyz="-0.145 -0.17 -0.0625" rpy="0 0 0"/>
     <geometry>
-      <mesh filename="package://mobile_description/meshes/front_left_wheel_1.stl" scale="0.001 0.001 0.001"/>
+      <mesh filename="file://$(find mobile_description)/meshes/front_left_wheel_1.stl" scale="0.001 0.001 0.001"/>
     </geometry>
   </collision>
@@ -93,5 +93,5 @@
     <origin xyz="0.145 -0.17 -0.0625" rpy="0 0 0"/>
     <geometry>
-      <mesh filename="package://mobile_description/meshes/rear_left_wheel_1.stl" scale="0.001 0.001 0.001"/>
+      <mesh filename="file://$(find mobile_description)/meshes/rear_left_wheel_1.stl" scale="0.001 0.001 0.001"/>
     </geometry>
     <material name="silver"/>
@@ -100,5 +100,5 @@
     <origin xyz="0.145 -0.17 -0.0625" rpy="0 0 0"/>
     <geometry>
-      <mesh filename="package://mobile_description/meshes/rear_left_wheel_1.stl" scale="0.001 0.001 0.001"/>
+      <mesh filename="file://$(find mobile_description)/meshes/rear_left_wheel_1.stl" scale="0.001 0.001 0.001"/>
     </geometry>
   </collision>
@@ -113,5 +113,5 @@
     <origin xyz="-0.205 -0.0 -0.3275" rpy="0 0 0"/>
     <geometry>
-      <mesh filename="package://mobile_description/meshes/lidar_1.stl" scale="0.001 0.001 0.001"/>
+      <mesh filename="file://$(find mobile_description)/meshes/lidar_1.stl" scale="0.001 0.001 0.001"/>
     </geometry>
     <material name="silver"/>
@@ -120,5 +120,5 @@
     <origin xyz="-0.205 -0.0 -0.3275" rpy="0 0 0"/>
     <geometry>
-      <mesh filename="package://mobile_description/meshes/lidar_1.stl" scale="0.001 0.001 0.001"/>
+      <mesh filename="file://$(find mobile_description)/meshes/lidar_1.stl" scale="0.001 0.001 0.001"/>
     </geometry>
   </collision>
@@ -133,5 +133,5 @@
     <origin xyz="-0.0 -0.0 -0.3275" rpy="0 0 0"/>
     <geometry>
-      <mesh filename="package://mobile_description/meshes/imu_1.stl" scale="0.001 0.001 0.001"/>
+      <mesh filename="file://$(find mobile_description)/meshes/imu_1.stl" scale="0.001 0.001 0.001"/>
     </geometry>
     <material name="silver"/>
@@ -140,5 +140,5 @@
     <origin xyz="-0.0 -0.0 -0.3275" rpy="0 0 0"/>
     <geometry>
-      <mesh filename="package://mobile_description/meshes/imu_1.stl" scale="0.001 0.001 0.001"/>
+      <mesh filename="file://$(find mobile_description)/meshes/imu_1.stl" scale="0.001 0.001 0.001"/>
     </geometry>
   </collision>
