Commit message: autogit

File: src/mobile_description/urdf/mobile.urdf (robot description, URDF)
Before this commit: robot mobile, 8 links, 7 joints
Joints:
- joint base_joint: axis (none) -> 0.0 0.0 0.0

Commit message: autogit

File: src/mobile_description/urdf/mobile.urdf (robot description, URDF)
Before this commit: robot mobile, 8 links, 7 joints
Joints:
- joint imu_joint: origin xyz=0.0 0.0 0.3275 rpy=0 0 0 -> xyz=0.0 0.0 0.220 rpy=0 0 0
- joint lidar_joint: origin xyz=0.205 0.0 0.3275 rpy=0 0 0 -> xyz=0.285 0 0.200 rpy=0 0 0

Commit message: autogit

File: src/mobile_description/urdf/mobile.urdf (robot description, URDF)
Before this commit: robot mobile, 8 links, 7 joints
Joints:
- joint front_left_joint: origin xyz=0.145 0.17 0.0625 rpy=0 0 0 -> xyz=0.240 0.22 0.0625 rpy=0 0 0
- joint front_right_joint: origin xyz=0.145 -0.17 0.0625 rpy=0 0 0 -> xyz=0.240 -0.22 0.0625 rpy=0 0 0
- joint rear_left_joint: origin xyz=-0.145 0.17 0.0625 rpy=0 0 0 -> xyz=-0.240 0.22 0.0625 rpy=0 0 0
- joint rear_right_joint: origin xyz=-0.145 -0.17 0.0625 rpy=0 0 0 -> xyz=-0.240 -0.22 0.0625 rpy=0 0 0

Commit message: autogit

File: src/mobile_description/urdf/mobile.urdf (robot description, URDF)
Before this commit: robot mobile, 8 links, 7 joints
Joints:
- joint lidar_joint: origin xyz=0.285 0 0.200 rpy=0 0 0 -> xyz=0.285 0 0.185 rpy=0 0 0
