Commit message: auto git from ubuntu

File: install/mobile_description/share/mobile_description/urdf/mobile.urdf (robot description, URDF)
Before this commit: robot mobile, 7 links, 6 joints
Links:
- added link base_footprint
Joints:
- added joint base_joint: type fixed, parent base_footprint, child base_link, origin xyz=0 0 0.005 rpy=0 0 0
